File: keychainProj.kicad_pcb (KiCad board)
At the start: 2 copper layers, 100 x 65.8 mm, 34 parts, among them J1 Conn_01x04_Pin, J2 USB_C_Receptacle_PowerOnly_6P, SW1 SW_SPDT_MSM, U1 AMS1117CD-3.3, U2 LIS3DH, U4 CH32V003FxPx

Commit message: Put thruholes on the back, smd all on front
Parts:
- BZ1, C4, U1: moved to F.Cu
- moved BZ1 6.37 mm to (160.7, 61.0), turned to 0 degrees
- moved U1 5.06 mm to (131.7, 101.8)
- moved C4 3.90 mm to (131.8, 93.0), turned to 90 degrees
Routing:
- net Net-(U1-VI): track 31.7 -> 22.2 mm, vias 1 -> 2
- net GND: track 178.2 -> 187.2 mm, vias 6 -> 7
- net Net-(SW1-4): track 77.1 -> 70.1 mm, vias 0 -> 1
- net Net-(BZ1-+): track 35.7 -> 37.9 mm
Other:
- board text removed: "+"
