File: PCB/keychainProj.kicad_pcb (KiCad board)
At the start: 2 copper layers, 100 x 65.8 mm, 34 parts, among them J1 Conn_01x04_Pin, J2 USB_C_Receptacle_PowerOnly_6P, SW1 SW_SPDT_MSM, U1 AMS1117CD-3.3, U2 LIS3DH, U4 CH32V003FxPx

Commit message: Simplified PCB and made for in depth bom files
Parts:
- removed SW1: SW_SPDT_MSM, Button_Switch_THT:SW_Slide_SPDT_Straight_CK_OS102011MS2Q
- added SW2: MST-12D18G4 SPDT SLIDE SWITCH, Newsymbols:SW-SMD_MST-12D18G4-SPDT-SLIDE-SWITCH, F.Cu at (190.0, 102.2)
- R5, R6: value 47 -> 0
- U2: footprint Package_LGA:LGA-16_3x3mm_P0.5mm_LayoutBorder3x5y -> ModuleLibrary:LIS3DH_Aliexpress_Module
- moved R9 10.6 mm to (200.8, 74.8)
- moved U2 10.6 mm to (202.5, 85.2), turned to 90 degrees
- moved R8 3.75 mm to (195.5, 85.5)
- moved R12 3.40 mm to (199.6, 82.2), turned to 180 degrees
Routing:
- net Net-(U2-INT1): track 22.6 -> 48.2 mm, vias 0 -> 1
- net Net-(U2-SPC): track 24.8 -> 39.1 mm, vias 3 -> 2
- net Net-(U2-SDI): track 29.5 -> 18.2 mm, vias 2 -> 0
- net Net-(BT1-+): track 48.4 -> 55.3 mm, vias 0 -> 1
- net Net-(U2-SDO): track 11.1 -> 4.67 mm
- net Net-(U4-PC3): track 121.6 -> 126.8 mm
- net +3.3V: track 152.3 -> 155.4 mm, vias 5 -> 6
- net GND: track 187.2 -> 184.9 mm, vias 7 -> 6
- net Net-(U4-PD2): track 33.9 -> 32.7 mm
- net Net-(U1-VO): track 70.1 -> 70.6 mm, vias 1 -> 2
Other:
- board text added: "USB BT"
- board text removed: "BT off USB"
